File: artix-pcie/fpga.sch (KiCad schematic (older format))
At the start: 3 parts, among them P1 JTAG_CONN, U1 xc7a15tfgg484, U2 N25Q256_QSPI

Commit message: working the hierarchy
Changed lines of the file:
@@
 EESchema Schematic File Version 2
+LIBS:artix-pcie-board-rescue
 LIBS:TOFE
 LIBS:xilinx7
@@
 	1    0    0    -1
 $EndComp
+Text HLabel 11750 7550 0    60   Input ~ 0
+PETp0
+Text HLabel 11750 7650 0    60   Input ~ 0
+PETn0
+Text HLabel 11750 8150 0    60   Input ~ 0
+PETp1
+Text HLabel 11750 8250 0    60   Input ~ 0
+PETn1
+Text HLabel 11750 8550 0    60   Input ~ 0
+PETp2
+Text HLabel 11750 8650 0    60   Input ~ 0
+PETn2
+Text HLabel 11750 8950 0    60   Input ~ 0
+PETp3
+Text HLabel 11750 9050 0    60   Input ~ 0
+PETn3
+Text HLabel 12550 7500 0    60   Input ~ 0
+REFCLK+
+Text HLabel 12550 7600 0    60   Input ~ 0
+REFCLK-
+Text HLabel 12550 7800 0    60   Output ~ 0
+PERp0
+Text HLabel 12550 7900 0    60   Output ~ 0
+PERn0
+Text HLabel 12550 8400 0    60   Output ~ 0
+PERp1
+Text HLabel 12550 8500 0    60   Output ~ 0
+PERn1
+Text HLabel 12550 8800 0    60   Output ~ 0
+PERp2
+Text HLabel 12550 8900 0    60   Output ~ 0
+PERn2
+Text HLabel 12550 9200 0    60   Output ~ 0
+PERp3
+Text HLabel 12550 9300 0    60   Output ~ 0
+PERn3
+Text HLabel 12550 7100 0    60   Input ~ 0
+PERST#
 $EndSCHEMATC
