File: artix-pcie/pcie.sch (KiCad schematic (older format))
At the start: 1 part, among them P2 TOFE-4X

Commit message: working the hierarchy
Connections:
- net PRSNT#: now reaches P2.A1 (~PRSNT1)
- net PRSNT#: now also P2.B31 (~PRSNT2)
- net PERST#: now reaches P2.A11 (PERST#)
- net pcie_refclk+ renamed REFCLK+
- net pcie_refclk- renamed REFCLK-
- no-connect marks 4 -> 17
Changed lines of the file:
@@
 EESchema Schematic File Version 2
+LIBS:artix-pcie-board-rescue
 LIBS:TOFE
 LIBS:xilinx7
@@
 U 1 1 5685ABCA
 P 4200 5150
+AR Path="/5685ABCA" Ref="P2"  Part="1"
+AR Path="/5685901C/5685ABCA" Ref="P2"  Part="1"
 F 0 "P2" H 3750 8137 60  0000 C CNN
 F 1 "TOFE-4X" H 3750 8031 60  0000 C CNN
@@
 Text HLabel 5850 6350 2    60   Output ~ 0
 GND
-Text HLabel 6150 3850 2    60   Output ~ 0
-pcie_refclk+
-Text HLabel 6150 3950 2    60   Output ~ 0
-pcie_refclk-
-Wire Wire Line
-	4600 3850 6150 3850
-Wire Wire Line
-	6150 3950 4600 3950
+Text HLabel 6350 3850 2    60   Output ~ 0
+REFCLK+
+Text HLabel 6350 3950 2    60   Output ~ 0
+REFCLK-
+Wire Wire Line
+	4600 3850 6350 3850
+Wire Wire Line
+	4600 3950 6350 3950
 Wire Wire Line
 	2900 3950 1500 3950
@@
 Text HLabel 6350 5650 2    60   Input ~ 0
 PERn3
+Wire Wire Line
+	2900 5750 2400 5750
+Wire Wire Line
+	2400 5750 2400 2000
+Wire Wire Line
+	2400 2000 4700 2000
+Wire Wire Line
+	4700 2000 4700 2450
+Wire Wire Line
+	4700 2450 4600 2450
+Text Label 3700 2000 0    60   ~ 0
+PRSNT#
+NoConn ~ 2900 4250
+NoConn ~ 2900 3750
+NoConn ~ 2900 5650
+NoConn ~ 4600 5850
+NoConn ~ 4600 4550
+NoConn ~ 4600 2850
+NoConn ~ 4600 2950
+NoConn ~ 4600 3050
+NoConn ~ 4600 3150
+NoConn ~ 2900 3250
+Text HLabel 6350 3450 2    60   Output ~ 0
+PERST#
+Wire Wire Line
+	4600 3450 6350 3450
+NoConn ~ 2900 2850
+NoConn ~ 2900 2950
+NoConn ~ 2900 3450
 $EndSCHEMATC

Commit message: fpga compiles and reports power. need to add pmod, oscillator and power supply
Changed lines of the file:
@@
 12V
 Wire Wire Line
-	6100 1850 2750 1850
+	6100 1850 4800 1850
 Wire Wire Line
-	2750 1850 2750 2650
+	4800 1850 2750 1850
+Wire Wire Line
+	2750 1850 2750 2450
+Wire Wire Line
+	2750 2450 2750 2550
+Wire Wire Line
+	2750 2550 2750 2650
 Wire Wire Line
 	2750 2650 2900 2650
@@
 	4800 2650 4600 2650
 Wire Wire Line
-	4800 1850 4800 2650
+	4800 1850 4800 2550
+Wire Wire Line
+	4800 2550 4800 2650
 Wire Wire Line
 	4800 2550 4600 2550
@@
 NoConn ~ 2900 3350
 Wire Wire Line
-	5850 6350 2600 6350
+	5850 6350 4950 6350
 Wire Wire Line
-	2600 6350 2600 2750
+	4950 6350 2600 6350
+Wire Wire Line
+	2600 6350 2600 5850
+Wire Wire Line
+	2600 5850 2600 5550
+Wire Wire Line
+	2600 5550 2600 5250
+Wire Wire Line
+	2600 5250 2600 5150
+Wire Wire Line
+	2600 5150 2600 4850
+Wire Wire Line
+	2600 4850 2600 4750
+Wire Wire Line
+	2600 4750 2600 4350
+Wire Wire Line
+	2600 4350 2600 4150
+Wire Wire Line
+	2600 4150 2600 3850
+Wire Wire Line
+	2600 3850 2600 3050
+Wire Wire Line
+	2600 3050 2600 2750
 Wire Wire Line
 	2600 2750 2900 2750
@@
 	4600 2750 4950 2750
 Wire Wire Line
-	4950 2750 4950 6350
+	4950 2750 4950 3750
+Wire Wire Line
+	4950 3750 4950 4050
+Wire Wire Line
+	4950 4050 4950 4350
+Wire Wire Line
+	4950 4350 4950 4650
+Wire Wire Line
+	4950 4650 4950 4950
+Wire Wire Line
+	4950 4950 4950 5050
+Wire Wire Line
+	4950 5050 4950 5350
+Wire Wire Line
+	4950 5350 4950 5450
+Wire Wire Line
+	4950 5450 4950 5750
+Wire Wire Line
+	4950 5750 4950 6350
 Connection ~ 4950 6350
 Wire Wire Line
